File: LattePanda_Module.kicad_sch (KiCad schematic)
At the start: 12 parts, among them J1 Conn_01x03_Pin

Commit message: added reference design and finished routing
Other:
- note added: "DDI/TCP functions are defined by the BIOS source code. Cannot be changed in BIOS settings. Before starting design, you should choose one of the available BIOS configurations on: https://github.com/LattePandaTeam/LattePanda-Mu The default functions are defined as follows: - DDIA: eDP 1.4b (the 40Pin connector on the Mu) - DDIB: HDMI 2.0 - TCP0: HDMI 2.0 - TCP1: USB TypeC (need external PD controll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"
- note added: "HSIO functions are defined by the BIOS source code, Cannot be changed in BIOS settings. Before starting design, you should choose one of the available BIOS configurations on: https://github.com/LattePandaTeam/LattePanda-Mu The default functions are defined as follows: - HSIO0: USB3.2 10Gbps - HSIO1: USB3.2 10Gbps - HSIO2: PCIe 3.0 x1 - HSIO3: PCIe 3.0 x1 - HSIO8: PCIe 3.0 x4 (Lane 0) - HSIO9: PCI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"
- note removed: "DDI/TCP functions are defined by the BIOS source code, Cannot be changed in BIOS settings. Before starting design, you should choose one of the available BIOS configurations on: https://github.com/LattePandaTeam/LattePanda-Mu The default functions are defined as follows: - DDIA: eDP 1.4b (the 40Pin connector on the Mu) - DDIB: HDMI 2.0 - TCP0: HDMI 2.0 - TCP1: USB TypeC (need external PD controll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"
- note removed: "HSIO functions are defined by the BIOS source code, Cannot be changed in BIOS settings. Before starting design, you should choose one of the available BIOS configurations on: https://github.com/LattePandaTeam/LattePanda-Mu Or contact techsupport for custom your BIOS The default functions are defined as follows: - HSIO0: USB3.2 10Gbps - HSIO1: USB3.2 10Gbps - HSIO2: PCIe 3.0 x1 - HSIO3: PCIe 3.0 x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"
Changed lines of the file:
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@@
 (kicad_sch
-	(version 20260101)
+	(version 20260306)
 	(generator "eeschema")
 	(generator_version "10.0")
@@
 	(text "Sleeping State Signal\n\n- SLS_S0: \n  - S0 (Working): HIGH\n  - S3 (Slpeeping): LOW\n  - S4 (Hibernation): LOW\n  - S5 (Soft Off): LOW\n- SLS_S3:\n  - S0 (Working): HIGH\n  - S3 (Slpeeping): HIGH\n  - S4 (Hibernation): LOW\n  - S5 (Soft Off): LOW"
 		(exclude_from_sim no)
-		(at 184.404 56.896 0)
+		(at 157.226 44.45 0)
 		(effects
 			(font
@@
 		)
 	)
-	(text "DDI/TCP functions are defined by the BIOS source code, \nCannot be changed in BIOS settings.\n\nBefore starting design, you should choose one of\nthe available BIOS configurations on:\nhttps://github.com/LattePandaTeam/LattePanda-Mu\n\nThe default functions are defined as follows:\n\n- DDIA: eDP 1.4b (the 40Pin connector on the Mu)\n\n- DDIB: HDMI 2.0\n\n- TCP0: HDMI 2.0\n\n- TCP1: USB TypeC (need external PD controller)"
+	(text "DDI/TCP functions are defined by the BIOS source code. \nCannot be changed in BIOS settings.\n\nBefore starting design, you should choose one of\nthe available BIOS configurations on:\nhttps://github.com/LattePandaTeam/LattePanda-Mu\n\nThe default functions are defined as follows:\n\n- DDIA: eDP 1.4b (the 40Pin connector on the Mu)\n\n- DDIB: HDMI 2.0\n\n- TCP0: HDMI 2.0\n\n- TCP1: USB TypeC (need external PD controller)"
 		(exclude_from_sim no)
 		(at 79.248 228.346 0)
@@
 		)
 	)
-	(text "HSIO functions are defined by the BIOS source code, \nCannot be changed in BIOS settings.\n\nBefore starting design, you should choose one of\nthe available BIOS configurations on:\nhttps://github.com/LattePandaTeam/LattePanda-Mu\nOr contact techsupport for custom your BIOS\n\nThe default functions are defined as follows:\n\n- HSIO0: USB3.2 10Gbps\n- HSIO1: USB3.2 10Gbps\n- HSIO2: PCIe 3.0 x1\n- HSIO3: PCIe 3.0 x1\n\n- HSIO8: PCIe 3.0 x4 (Lane 0)\n- HSIO9: PCIe 3.0 x4 (Lane 1)\n- HSIO10: PCIe 3.0 x4 (Lane 2)\n- HSIO11: PCIe 3.0 x4 (Lane 3)\n\n- HSIO6: PCIe 3.0 x1"
+	(text "HSIO functions are defined by the BIOS source code, \nCannot be changed in BIOS settings.\n\nBefore starting design, you should choose one of\nthe available BIOS configurations on:\nhttps://github.com/LattePandaTeam/LattePanda-Mu\n\nThe default functions are defined as follows:\n\n- HSIO0: USB3.2 10Gbps\n- HSIO1: USB3.2 10Gbps\n- HSIO2: PCIe 3.0 x1\n- HSIO3: PCIe 3.0 x1\n\n- HSIO8: PCIe 3.0 x4 (Lane 0)\n- HSIO9: PCIe 3.0 x4 (Lane 1)\n- HSIO10: PCIe 3.0 x4 (Lane 2)\n- HSIO11: PCIe 3.0 x4 (Lane 3)\n\n- HSIO6: PCIe 3.0 x1"
 		(exclude_from_sim no)
 		(at 79.248 101.346 0)
@@
 		)
 	)
+	(hierarchical_label "HSIO_10_RX-"
+		(shape input)
+		(at 472.44 153.67 180)
+		(effects
+			(font
+				(size 1.27 1.27)
+			)
+			(justify right)
+		)
+	)
 	(hierarchical_label "DDI_B_TX0+"
 		(shape output)
@@
 		)
 	)
+	(hierarchical_label "HSIO_10_RX+"
+		(shape input)
+		(at 472.44 151.13 180)
+		(effects
+			(font
+				(size 1.27 1.27)
+			)
+			(justify right)
+		)
+	)
 	(hierarchical_label "HSIO_9_TX+"
 		(shape output)
@@
 		)
 	)
+	(hierarchical_label "HSIO_11_RX+"
+		(shape input)
+		(at 472.44 161.29 180)
+		(effects
+			(font
+				(size 1.27 1.27)
+			)
+			(justify right)
+		)
+	)
 	(hierarchical_label "USB_2_P7-"
 		(shape bidirectional)
@@
 		)
 	)
+	(hierarchical_label "HSIO_11_RX-"
+		(shape input)
+		(at 472.44 163.83 180)
+		(effects
+			(font
+				(size 1.27 1.27)
+			)
+			(justify right)
+		)
+	)
 	(hierarchical_label "DDI_B_DDC_SCL"
 		(shape output)
@@
 		)
 		(instances
-			(project ""
+			(project "LattePandaMu_carrier_custom"
 				(path "/8a2b43cc-acba-4686-85d9-5be8ade4e79b/4ee1a750-9135-4964-a1b8-1eecfd9d94af"
 					(reference "BT1")
@@
 		)
 		(instances
-			(project ""
+			(project "LattePandaMu_carrier_custom"
 				(path "/8a2b43cc-acba-4686-85d9-5be8ade4e79b/4ee1a750-9135-4964-a1b8-1eecfd9d94af"
 					(reference "#PWR015")
@@
 		)
 		(instances
-			(project ""
+			(project "LattePandaMu_carrier_custom"
 				(path "/8a2b43cc-acba-4686-85d9-5be8ade4e79b/4ee1a750-9135-4964-a1b8-1eecfd9d94af"
 					(reference "TP7")
@@
 		)
 		(instances
-			(project ""
+			(project "LattePandaMu_carrier_custom"
 				(path "/8a2b43cc-acba-4686-85d9-5be8ade4e79b/4ee1a750-9135-4964-a1b8-1eecfd9d94af"
 					(reference "R2")
@@
 		)
 		(instances
-			(project ""
+			(project "LattePandaMu_carrier_custom"
 				(path "/8a2b43cc-acba-4686-85d9-5be8ade4e79b/4ee1a750-9135-4964-a1b8-1eecfd9d94af"
 					(reference "#PWR05")
@@
 		)
 		(instances
-			(project ""
+			(project "LattePandaMu_carrier_custom"
 				(path "/8a2b43cc-acba-4686-85d9-5be8ade4e79b/4ee1a750-9135-4964-a1b8-1eecfd9d94af"
 					(reference "J1")
@@
 		)
 		(instances
-			(project ""
+			(project "LattePandaMu_carrier_custom"
 				(path "/8a2b43cc-acba-4686-85d9-5be8ade4e79b/4ee1a750-9135-4964-a1b8-1eecfd9d94af"
 					(reference "#PWR013")
@@
 		)
 		(instances
-			(project ""
+			(project "LattePandaMu_carrier_custom"
 				(path "/8a2b43cc-acba-4686-85d9-5be8ade4e79b/4ee1a750-9135-4964-a1b8-1eecfd9d94af"
 					(reference "#PWR07")
@@
 		)
 		(instances
-			(project ""
+			(project "LattePandaMu_carrier_custom"
 				(path "/8a2b43cc-acba-4686-85d9-5be8ade4e79b/4ee1a750-9135-4964-a1b8-1eecfd9d94af"
 					(reference "#PWR012")
@@
 		)
 		(instances
-			(project ""
+			(project "LattePandaMu_carrier_custom"
 				(path "/8a2b43cc-acba-4686-85d9-5be8ade4e79b/4ee1a750-9135-4964-a1b8-1eecfd9d94af"
 					(reference "#PWR010")
@@
 		)
 		(instances
-			(project ""
+			(project "LattePandaMu_carrier_custom"
 				(path "/8a2b43cc-acba-4686-85d9-5be8ade4e79b/4ee1a750-9135-4964-a1b8-1eecfd9d94af"
 					(reference "#PWR011")
@@
 		)
 		(instances
-			(project ""
+			(project "LattePandaMu_carrier_custom"
 				(path "/8a2b43cc-acba-4686-85d9-5be8ade4e79b/4ee1a750-9135-4964-a1b8-1eecfd9d94af"
 					(reference "H5")
@@
 		)
 		(instances
-			(project ""
+			(project "LattePandaMu_carrier_custom"
 				(path "/8a2b43cc-acba-4686-85d9-5be8ade4e79b/4ee1a750-9135-4964-a1b8-1eecfd9d94af"
 					(reference "#PWR06")
@@
 		)
 		(instances
-			(project ""
+			(project "LattePandaMu_carrier_custom"
 				(path "/8a2b43cc-acba-4686-85d9-5be8ade4e79b/4ee1a750-9135-4964-a1b8-1eecfd9d94af"
 					(reference "A1")
@@
 		)
 		(instances
-			(project ""
+			(project "LattePandaMu_carrier_custom"
 				(path "/8a2b43cc-acba-4686-85d9-5be8ade4e79b/4ee1a750-9135-4964-a1b8-1eecfd9d94af"
 					(reference "#PWR09")
@@
 		)
 		(instances
-			(project ""
+			(project "LattePandaMu_carrier_custom"
 				(path "/8a2b43cc-acba-4686-85d9-5be8ade4e79b/4ee1a750-9135-4964-a1b8-1eecfd9d94af"
 					(reference "#FLG01")
