File: ethernet.kicad_sch (KiCad schematic)
At the start: 27 parts, among them J6 RJ45_RB1-125B8G1A, U6 RTL8111H-CG-RH, U7 D3V3XA4B10LP, U8 D3V3XA4B10LP, Y1 25MHz

Commit message: added reference design and finished routing
Other:
- moved on the sheet: C33, C34, C35, C36, C37, C38, C39, C40, C41, C42, C43, C44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
