File: psu.kicad_sch (KiCad schematic)
At the start: 87 parts, among them J17 Barrel_Jack_Switch, J18 USB_C_Receptacle_USB2.0_16P, Q5 2N7002, Q6 2N7002, Q7 AON7262E, Q8 2N7002, SW1 SW_Push, SW2 SW_Push, U13 TL431DBZ, U14 USB PD等快充协议受电芯片-CH224K-ESSOP10, U15 LM2734X, U16 LM2734X

Commit message: added reference design and finished routing
Connections:
- net SLS_S3 is gone; now on net VDC: JP1.3 (B)
- net GND: now also C65.1, C68.1; no longer C65.2, C68.2
- net VDC: now also C65.2, C68.2, JP1.2 (C), R46.2; no longer C65.1, C68.1
Other:
- moved on the sheet: C62, C63, C64, C67, D22, D23, D24, JP1, Q5, Q6, Q7, Q8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
