File: LattePandaMu_carrier_custom.kicad_pcb (KiCad board)
At the start: 4 copper layers, 170.1 x 100 mm, 220 parts, among them J1 Conn_01x03_Pin, J10 Conn_01x03_Pin, J11 Conn_01x03_Pin, J12 Conn_01x04_Pin, J13 Conn_01x04_Pin, J14 Conn_01x03_Pin, J15 Bus_M.2_Socket_M, J16 Bus_M.2_Socket_E, J17 Barrel_Jack_Switch, J18 USB_C_Receptacle_USB2.0_16P, J19 Conn_01x04_Pin, J20 Conn_01x04_Pin, J21 Conn_01x04_Pin, J3 HDMI_A, J4 USB3_A_Stacked, J5 USB_A_Stacked, J6 RJ45_RB1-125B8G1A, J7 Conn_01x04_Pin, J8 Conn_01x03_Pin, J9 Conn_01x04_Pin, M1 Fan_4pin, Q1 2N7002, Q2 2SK3018, Q3 2SK3018, Q4 2SK3018, Q8 2N7002, SW1 SW_Push, SW2 SW_Push, U1 D3V3XA4B10LP, U10 ULC0524P, U11 ULC0524P, U12 ULC0524P, U14 USB PD-CH224K-ESSOP10, U15 LM2734X, U16 LM2734X, U17 ULC0524P, U2 D3V3XA4B10LP, U3 D3V3XA4B10LP, U4 D3V3XA4B10LP, U5 D3V3XA4B10LP, U6 RTL8111H-CG-RH, U7 D3V3XA4B10LP, U8 D3V3XA4B10LP, U9 ULC0524P, Y1 25MHz

Commit message: improved layout
Parts:
- removed G***: LOGO, Logo:TE_Logo_footprint_15mm
- removed REF**: KiCad-Logo2_5mm_SilkScreen, Symbol:KiCad-Logo2_5mm_SilkScreen
- removed REF**: OSHW-Logo_5.7x6mm_SilkScreen, Symbol:OSHW-Logo_5.7x6mm_SilkScreen
Other:
- board text removed: "LattePanda Mu Tech Explorations Custom Board V1"
