File: pciex4.kicad_sch (KiCad schematic)
At the start: 17 parts, among them J2 Bus_PCI_Express_x4

Commit message: added pcie to schematic
Parts:
- C1, C10, C11, C13, C14, C15, C16, C2, C3, C4, C5, C6, C7, C8, C9, J2, TP1: now fitted
Changed lines of the file:
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@@
 		(exclude_from_sim no)
 		(in_bom yes)
-		(on_board no)
-		(in_pos_files yes)
-		(dnp yes)
+		(on_board yes)
+		(in_pos_files yes)
+		(dnp no)
 		(property "Reference" "C3"
 			(at 114.935 118.11 90)
@@
 		(exclude_from_sim no)
 		(in_bom yes)
-		(on_board no)
-		(in_pos_files yes)
-		(dnp yes)
+		(on_board yes)
+		(in_pos_files yes)
+		(dnp no)
 		(property "Reference" "C8"
 			(at 114.935 130.81 90)
@@
 		(exclude_from_sim no)
 		(in_bom yes)
-		(on_board no)
-		(in_pos_files yes)
-		(dnp yes)
+		(on_board yes)
+		(in_pos_files yes)
+		(dnp no)
 		(fields_autoplaced yes)
 		(property "Reference" "#PWR060"
@@
 		(exclude_from_sim no)
 		(in_bom yes)
-		(on_board no)
-		(in_pos_files yes)
-		(dnp yes)
+		(on_board yes)
+		(in_pos_files yes)
+		(dnp no)
 		(property "Reference" "C10"
 			(at 116.84 65.405 0)
@@
 		(exclude_from_sim no)
 		(in_bom yes)
-		(on_board no)
-		(in_pos_files yes)
-		(dnp yes)
+		(on_board yes)
+		(in_pos_files yes)
+		(dnp no)
 		(fields_autoplaced yes)
 		(property "Reference" "J2"
@@
 		(exclude_from_sim no)
 		(in_bom yes)
-		(on_board no)
-		(in_pos_files yes)
-		(dnp yes)
+		(on_board yes)
+		(in_pos_files yes)
+		(dnp no)
 		(property "Reference" "C5"
 			(at 114.935 123.19 90)
@@
 		(exclude_from_sim no)
 		(in_bom yes)
-		(on_board no)
-		(in_pos_files yes)
-		(dnp yes)
+		(on_board yes)
+		(in_pos_files yes)
+		(dnp no)
 		(property "Reference" "C1"
 			(at 114.935 113.03 90)
@@
 		(exclude_from_sim no)
 		(in_bom yes)
-		(on_board no)
-		(in_pos_files yes)
-		(dnp yes)
+		(on_board yes)
+		(in_pos_files yes)
+		(dnp no)
 		(fields_autoplaced yes)
 		(property "Reference" "#PWR056"
@@
 		(exclude_from_sim no)
 		(in_bom yes)
-		(on_board no)
-		(in_pos_files yes)
-		(dnp yes)
+		(on_board yes)
+		(in_pos_files yes)
+		(dnp no)
 		(property "Reference" "C11"
 			(at 127.635 65.405 0)
@@
 		(exclude_from_sim no)
 		(in_bom yes)
-		(on_board no)
-		(in_pos_files yes)
-		(dnp yes)
+		(on_board yes)
+		(in_pos_files yes)
+		(dnp no)
 		(property "Reference" "C13"
 			(at 147.955 43.18 0)
@@
 		(exclude_from_sim no)
 		(in_bom yes)
-		(on_board no)
-		(in_pos_files yes)
-		(dnp yes)
+		(on_board yes)
+		(in_pos_files yes)
+		(dnp no)
 		(property "Reference" "C2"
 			(at 114.935 115.57 90)
@@
 		(exclude_from_sim no)
 		(in_bom yes)
-		(on_board no)
-		(in_pos_files yes)
-		(dnp yes)
+		(on_board yes)
+		(in_pos_files yes)
+		(dnp no)
 		(property "Reference" "C15"
 			(at 173.99 65.405 0)
@@
 		(exclude_from_sim no)
 		(in_bom yes)
-		(on_board no)
-		(in_pos_files yes)
-		(dnp yes)
+		(on_board yes)
+		(in_pos_files yes)
+		(dnp no)
 		(property "Reference" "C14"
 			(at 154.305 43.18 0)
@@
 		(exclude_from_sim no)
 		(in_bom yes)
-		(on_board no)
-		(in_pos_files yes)
-		(dnp yes)
+		(on_board yes)
+		(in_pos_files yes)
+		(dnp no)
 		(fields_autoplaced yes)
 		(property "Reference" "#PWR0122"
@@
 		(exclude_from_sim no)
 		(in_bom yes)
-		(on_board no)
-		(in_pos_files yes)
-		(dnp yes)
+		(on_board yes)
+		(in_pos_files yes)
+		(dnp no)
 		(property "Reference" "C9"
 			(at 111.125 65.405 0)
@@
 		(exclude_from_sim no)
 		(in_bom yes)
-		(on_board no)
-		(in_pos_files yes)
-		(dnp yes)
+		(on_board yes)
+		(in_pos_files yes)
+		(dnp no)
 		(fields_autoplaced yes)
 		(property "Reference" "#PWR059"
@@
 		(exclude_from_sim no)
 		(in_bom yes)
-		(on_board no)
-		(in_pos_files yes)
-		(dnp yes)
+		(on_board yes)
+		(in_pos_files yes)
+		(dnp no)
 		(property "Reference" "C4"
 			(at 114.935 120.65 90)
@@
 		(exclude_from_sim no)
 		(in_bom yes)
-		(on_board no)
-		(in_pos_files yes)
-		(dnp yes)
+		(on_board yes)
+		(in_pos_files yes)
+		(dnp no)
 		(property "Reference" "C7"
 			(at 114.935 128.27 90)
@@
 		(exclude_from_sim no)
 		(in_bom yes)
-		(on_board no)
-		(in_pos_files yes)
-		(dnp yes)
+		(on_board yes)
+		(in_pos_files yes)
+		(dnp no)
 		(fields_autoplaced yes)
 		(property "Reference" "TP1"
@@
 		(exclude_from_sim no)
 		(in_bom yes)
-		(on_board no)
-		(in_pos_files yes)
-		(dnp yes)
+		(on_board yes)
+		(in_pos_files yes)
+		(dnp no)
 		(property "Reference" "C16"
 			(at 184.785 64.77 0)
@@
 		(exclude_from_sim no)
 		(in_bom yes)
-		(on_board no)
-		(in_pos_files yes)
-		(dnp yes)
+		(on_board yes)
+		(in_pos_files yes)
+		(dnp no)
 		(fields_autoplaced yes)
 		(property "Reference" "#PWR057"
@@
 		(exclude_from_sim no)
 		(in_bom yes)
-		(on_board no)
-		(in_pos_files yes)
-		(dnp yes)
+		(on_board yes)
+		(in_pos_files yes)
+		(dnp no)
 		(property "Reference" "C6"
 			(at 114.935 125.73 90)
@@
 		(exclude_from_sim no)
 		(in_bom yes)
-		(on_board no)
-		(in_pos_files yes)
-		(dnp yes)
+		(on_board yes)
+		(in_pos_files yes)
+		(dnp no)
 		(fields_autoplaced yes)
 		(property "Reference" "#PWR061"
@@
 		(exclude_from_sim no)
 		(in_bom yes)
-		(on_board no)
-		(in_pos_files yes)
-		(dnp yes)
+		(on_board yes)
+		(in_pos_files yes)
+		(dnp no)
 		(fields_autoplaced yes)
 		(property "Reference" "#PWR058"
